Commit message: tested on Go1 payload; 1m/s achieved

File: legged_examples/legged_unitree/legged_unitree_description/urdf/go1_payload.urdf (robot description, URDF)
Before this commit: robot robot, 19 links, 18 joints
Links:
- link unitree_payload: mass 2 -> 2.5
Joints:
- joint unitree_payload_joint: origin xyz=0.08 0. 0.11 rpy=0. 0. 0. -> xyz=0.10 0. 0.11 rpy=0. 0. 0.
